File: HW/PCB/60pc_pcb.kicad_pcb (KiCad board)
At the start: 2 copper layers, 306.5 x 98.2 mm, 153 parts, among them J1 USB_mini_micro_B, K1 KEYSW, K10 KEYSW, K11 KEYSW, K12 KEYSW, K13 KEYSW, K14 KEYSW, K15 KEYSW, K16 KEYSW, K17 KEYSW, K18 KEYSW, K19 KEYSW, K2 KEYSW, K21 KEYSW, K22 KEYSW, K23 KEYSW, K24 KEYSW, K26 KEYSW, K27 KEYSW, K28 KEYSW, K29 KEYSW, K3 KEYSW, K31 KEYSW, K32 KEYSW, K33 KEYSW, K34 KEYSW, K35 KEYSW, K36 KEYSW, K37 KEYSW, K38 KEYSW, K39 KEYSW, K4 KEYSW, K41 KEYSW, K42 KEYSW, K43 KEYSW, K44 KEYSW, K46 KEYSW, K47 KEYSW, K48 KEYSW, K49 KEYSW, K5 KEYSW, K51 KEYSW, K52 KEYSW, K53 KEYSW, K54 KEYSW, K55 KEYSW, K56 KEYSW, K57 KEYSW, K58 KEYSW, K59 KEYSW, K6 KEYSW, K60 KEYSW, K61 KEYSW, K62 KEYSW, K63 KEYSW, K64 KEYSW, K65 KEYSW, K66 KEYSW, K67 KEYSW, K68 KEYSW, K69 KEYSW, K7 KEYSW, K70 KEYSW, K71 KEYSW, K72 KEYSW, K74 KEYSW, K75 KEYSW, K8 KEYSW, K9 KEYSW, SW1 SW_PUSH, U1 ATMEGA32U4, Y1 Crystal_GND24

Commit message: Added M4 mounting holes to pcb
Parts:
- added REF**: MountingHole_4.3mm_M4_ISO7380_Pad, Mounting_Holes:MountingHole_4.3mm_M4_ISO7380_Pad, F.Cu at (374.0, 29.2)
- added REF**: MountingHole_4.3mm_M4_ISO7380_Pad, Mounting_Holes:MountingHole_4.3mm_M4_ISO7380_Pad, F.Cu at (374.0, 133.8)
- added REF**: MountingHole_4.3mm_M4_ISO7380_Pad, Mounting_Holes:MountingHole_4.3mm_M4_ISO7380_Pad, F.Cu at (86.2, 29.2)
- added REF**: MountingHole_4.3mm_M4_ISO7380_Pad, Mounting_Holes:MountingHole_4.3mm_M4_ISO7380_Pad, F.Cu at (90.5, 134.2)
- moved J1 7.85 mm to (97.8, 30.2)
Routing:
- net Net-(J1-Pad3): track 6.95 -> 14.8 mm
- net Net-(J1-Pad2): track 6.65 -> 14.5 mm
- net VCC: track 238.8 -> 246.7 mm
- net GND: track 226.5 -> 230.0 mm
Other:
- board size 306.5 x 98.2 mm -> 306.5 x 116 mm
