File: HW/PCB/60pc_pcb.kicad_v1.1_pcb.kicad_pcb (KiCad board)
At the start: 2 copper layers, 306.5 x 116 mm, 157 parts, among them J1 USB_mini_micro_B, K1 KEYSW, K10 KEYSW, K11 KEYSW, K12 KEYSW, K13 KEYSW, K14 KEYSW, K15 KEYSW, K16 KEYSW, K17 KEYSW, K18 KEYSW, K19 KEYSW, K2 KEYSW, K21 KEYSW, K22 KEYSW, K23 KEYSW, K24 KEYSW, K26 KEYSW, K27 KEYSW, K28 KEYSW, K29 KEYSW, K3 KEYSW, K31 KEYSW, K32 KEYSW, K33 KEYSW, K34 KEYSW, K35 KEYSW, K36 KEYSW, K37 KEYSW, K38 KEYSW, K39 KEYSW, K4 KEYSW, K41 KEYSW, K42 KEYSW, K43 KEYSW, K44 KEYSW, K46 KEYSW, K47 KEYSW, K48 KEYSW, K49 KEYSW, K5 KEYSW, K51 KEYSW, K52 KEYSW, K53 KEYSW, K54 KEYSW, K55 KEYSW, K56 KEYSW, K57 KEYSW, K58 KEYSW, K59 KEYSW, K6 KEYSW, K60 KEYSW, K61 KEYSW, K62 KEYSW, K63 KEYSW, K64 KEYSW, K65 KEYSW, K66 KEYSW, K67 KEYSW, K68 KEYSW, K69 KEYSW, K7 KEYSW, K70 KEYSW, K71 KEYSW, K72 KEYSW, K74 KEYSW, K75 KEYSW, K8 KEYSW, K9 KEYSW, SW1 SW_PUSH, U1 ATMEGA32U4, Y1 Crystal_GND24

Commit message: Version 1.1 edits
Smaller form factor.
4x M4 screws to 5x M2 screws.
Screws now placed between switched.
Dufferential routing return path and impedance matching improved.
Parts:
- removed the REF** at (374.0, 29.2)
- removed the REF** at (374.0, 133.8)
- removed the REF** at (86.2, 29.2)
- removed the REF** at (90.5, 134.2)
- added REF**: MountingHole_2.2mm_M2_ISO7380_Pad, Mounting_Holes:MountingHole_2.2mm_M2_ISO7380_Pad, F.Cu at (82.8, 53.0)
- added REF**: MountingHole_2.2mm_M2_ISO7380_Pad, Mounting_Holes:MountingHole_2.2mm_M2_ISO7380_Pad, F.Cu at (126.2, 110.0)
- added REF**: MountingHole_2.2mm_M2_ISO7380_Pad, Mounting_Holes:MountingHole_2.2mm_M2_ISO7380_Pad, F.Cu at (364.2, 52.5)
- added REF**: MountingHole_2.2mm_M2_ISO7380_Pad, Mounting_Holes:MountingHole_2.2mm_M2_ISO7380_Pad, F.Cu at (345.2, 110.0)
- added REF**: MountingHole_2.2mm_M2_ISO7380_Pad, Mounting_Holes:MountingHole_2.2mm_M2_ISO7380_Pad, F.Cu at (226.2, 72.0)
- moved J1 8.00 mm to (97.5, 38.2)
Routing:
- net GND: track 385.1 -> 344.4 mm, vias 16 -> 30
- net VCC: track 251.3 -> 242.6 mm
- net Net-(J1-Pad3): track 36.2 -> 28.3 mm
- net Net-(J1-Pad2): track 36.3 -> 28.3 mm
- net /Col0: track 176.5 -> 180.7 mm
- net /Row4: track 414.7 -> 416.0 mm
- net /Row3: track 424.4 -> 425.7 mm
- net /Row2: track 455.7 -> 456.9 mm
- net /Row1: track 479.1 -> 480.3 mm
- net /Row0: track 503.9 -> 505.2 mm
Other:
- board size 306.5 x 116 mm -> 306.8 x 98.5 mm

Commit message: Added Usb hole to v1.1
Routing:
- net GND: track 344.4 -> 210.5 mm, vias 30 -> 12
- net (no net): track 0.00 -> 133.8 mm, vias 1 -> 19
Changed lines of the file:
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@@
     (area 67.883333 28.8808 384.575001 131.5561)
     (thickness 1.6)
-    (drawings 20)
+    (drawings 22)
     (tracks 1163)
     (zones 0)
@@
   (layers
     (0 F.Cu signal)
-    (31 B.Cu signal hide)
+    (31 B.Cu signal)
     (32 B.Adhes user)
     (33 F.Adhes user)
     (34 B.Paste user)
     (35 F.Paste user)
-    (36 B.SilkS user hide)
-    (37 F.SilkS user hide)
+    (36 B.SilkS user)
+    (37 F.SilkS user)
     (38 B.Mask user)
     (39 F.Mask user)
-    (40 Dwgs.User user hide)
-    (41 Cmts.User user hide)
-    (42 Eco1.User user hide)
-    (43 Eco2.User user hide)
-    (44 Edge.Cuts user hide)
+    (40 Dwgs.User user)
+    (41 Cmts.User user)
+    (42 Eco1.User user)
+    (43 Eco2.User user)
+    (44 Edge.Cuts user)
     (45 Margin user hide)
     (46 B.CrtYd user)
@@
     (pad 1 thru_hole circle (at 0 0) (size 3.5 3.5) (drill 2.2) (layers *.Cu *.Mask))
   )
+  (dimension 306.75 (width 0.3) (layer Dwgs.User)
+    (gr_text "306.750 mm" (at 231.125 26.65) (layer Dwgs.User)
+      (effects (font (size 1.5 1.5) (thickness 0.3)))
+    )
+    (feature1 (pts (xy 77.75 31.75) (xy 77.75 25.3)))
+    (feature2 (pts (xy 384.5 31.75) (xy 384.5 25.3)))
+    (crossbar (pts (xy 384.5 28) (xy 77.75 28)))
+    (arrow1a (pts (xy 77.75 28) (xy 78.876504 27.413579)))
+    (arrow1b (pts (xy 77.75 28) (xy 78.876504 28.586421)))
+    (arrow2a (pts (xy 384.5 28) (xy 383.373496 27.413579)))
+    (arrow2b (pts (xy 384.5 28) (xy 383.373496 28.586421)))
+  )
+  (dimension 98.5 (width 0.3) (layer Dwgs.User)
+    (gr_text "98.500 mm" (at 391.1 81 270) (layer Dwgs.User)
+      (effects (font (size 1.5 1.5) (thickness 0.3)))
+    )
+    (feature1 (pts (xy 384.5 130.25) (xy 392.45 130.25)))
+    (feature2 (pts (xy 384.5 31.75) (xy 392.45 31.75)))
+    (crossbar (pts (xy 389.75 31.75) (xy 389.75 130.25)))
+    (arrow1a (pts (xy 389.75 130.25) (xy 389.163579 129.123496)))
+    (arrow1b (pts (xy 389.75 130.25) (xy 390.336421 129.123496)))
+    (arrow2a (pts (xy 389.75 31.75) (xy 389.163579 32.876504)))
+    (arrow2b (pts (xy 389.75 31.75) (xy 390.336421 32.876504)))
+  )
   (gr_line (start 380.5 130.25) (end 378 130.25) (angle 90) (layer Edge.Cuts) (width 0.15))
   (gr_line (start 381.75 31.75) (end 381.25 31.75) (angle 90) (layer Edge.Cuts) (width 0.15))
@@
   (gr_arc (start 381.75 34.5) (end 381.75 31.75) (angle 90) (layer Edge.Cuts) (width 0.15))
   (via (at 182.5 129) (size 0.6) (drill 0.4) (layers F.Cu B.Cu) (net 0))
-  (segment (start 95.9 38.25) (end 95.9 47.9) (width 0.25) (layer B.Cu) (net 1) (status 400000))
+  (segment (start 97.25 42.75) (end 97.25 48.136398) (width 0.25) (layer B.Cu) (net 0))
+  (via (at 96.75 40.75) (size 0.6) (drill 0.4) (layers F.Cu B.Cu) (net 0))
+  (segment (start 96.75 40.75) (end 97.25 41.25) (width 0.25) (layer B.Cu) (net 0))
+  (segment (start 97.25 41.25) (end 97.25 42.75) (width 0.25) (layer B.Cu) (net 0))
+  (via (at 177.5 105.25) (size 0.6) (drill 0.4) (layers F.Cu B.Cu) (net 0))
+  (segment (start 177.75 105) (end 177.5 105.25) (width 0.25) (layer B.Cu) (net 0))
+  (segment (start 177.75 94.5) (end 177.75 105) (width 0.25) (layer B.Cu) (net 0))
+  (segment (start 169 85.75) (end 177.75 94.5) (width 0.25) (layer B.Cu) (net 0))
+  (segment (start 169 75) (end 169 85.75) (width 0.25) (layer B.Cu) (net 0))
+  (segment (start 166.450002 72.450002) (end 169 75) (width 0.25) (layer B.Cu) (net 0))
+  (segment (start 108.700002 72.450002) (end 166.450002 72.450002) (width 0.25) (layer B.Cu) (net 0))
+  (segment (start 102.75 66.5) (end 108.700002 72.450002) (width 0.25) (layer B.Cu) (net 0))
+  (segment (start 102.75 61.5) (end 102.75 66.5) (width 0.25) (layer B.Cu) (net 0))
+  (segment (start 105 59.25) (end 102.75 61.5) (width 0.25) (layer B.Cu) (net 0))
+  (segment (start 105 55.886398) (end 105 59.25) (width 0.25) (layer B.Cu) (net 0))
+  (segment (start 97.25 48.136398) (end 105 55.886398) (width 0.25) (layer B.Cu) (net 0))
+  (via (at 144.5 69.75) (size 0.6) (drill 0.4) (layers F.Cu B.Cu) (net 0))
+  (via (at 149.25 74.5) (size 0.6) (drill 0.4) (layers F.Cu B.Cu) (net 0))
+  (via (at 162.25 69.75) (size 0.6) (drill 0.4) (layers F.Cu B.Cu) (net 0))
+  (via (at 158.25 69.75) (size 0.6) (drill 0.4) (layers F.Cu B.Cu) (net 0))
+  (via (at 141 69.75) (size 0.6) (drill 0.4) (layers F.Cu B.Cu) (net 0))
+  (via (at 130.25 74.5) (size 0.6) (drill 0.4) (layers F.Cu B.Cu) (net 0))
+  (via (at 125.25 69.75) (size 0.6) (drill 0.4) (layers F.Cu B.Cu) (net 0))
+  (via (at 126.75 74.5) (size 0.6) (drill 0.4) (layers F.Cu B.Cu) (net 0))
+  (via (at 122.5 69.75) (size 0.6) (drill 0.4) (layers F.Cu B.Cu) (net 0))
+  (via (at 153.75 117) (size 0.6) (drill 0.4) (layers F.Cu B.Cu) (net 0))
+  (via (at 159 106) (size 0.6) (drill 0.4) (layers F.Cu B.Cu) (net 0))
+  (via (at 158.75 92.25) (size 0.6) (drill 0.4) (layers F.Cu B.Cu) (net 0))
+  (via (at 145.75 74.5) (size 0.6) (drill 0.4) (layers F.Cu B.Cu) (net 0))
+  (via (at 146.25 116.75) (size 0.6) (drill 0.4) (layers F.Cu B.Cu) (net 0))
+  (via (at 141.25 108.75) (size 0.6) (drill 0.4) (layers F.Cu B.Cu) (net 0))
+  (via (at 141.25 92.25) (size 0.6) (drill 0.4) (layers F.Cu B.Cu) (net 0))
+  (segment (start 95.9 38.25) (end 95.9 47.9) (width 0.25) (layer B.Cu) (net 1))
   (segment (start 95.9 47.9) (end 96 48) (width 0.25) (layer B.Cu) (net 1))
   (segment (start 168.25 75.25) (end 168.25 87) (width 0.25) (layer B.Cu) (net 1))
@@
   (segment (start 180.5825 126.5825) (end 180.625 126.625) (width 0.25) (layer B.Cu) (net 1))
   (segment (start 183.0875 115.75) (end 183.0825 115.755) (width 0.25) (layer B.Cu) (net 1))
-  (segment (start 97.25 42.75) (end 97.25 48.136398) (width 0.25) (layer B.Cu) (net 2))
-  (via (at 96.75 40.75) (size 0.6) (drill 0.4) (layers F.Cu B.Cu) (net 2))
-  (segment (start 96.75 40.75) (end 97.25 41.25) (width 0.25) (layer B.Cu) (net 2))
-  (segment (start 97.25 41.25) (end 97.25 42.75) (width 0.25) (layer B.Cu) (net 2))
-  (via (at 177.5 105.25) (size 0.6) (drill 0.4) (layers F.Cu B.Cu) (net 2))
-  (segment (start 177.75 105) (end 177.5 105.25) (width 0.25) (layer B.Cu) (net 2))
-  (segment (start 177.75 94.5) (end 177.75 105) (width 0.25) (layer B.Cu) (net 2))
-  (segment (start 169 85.75) (end 177.75 94.5) (width 0.25) (layer B.Cu) (net 2))
-  (segment (start 169 75) (end 169 85.75) (width 0.25) (layer B.Cu) (net 2))
-  (segment (start 166.450002 72.450002) (end 169 75) (width 0.25) (layer B.Cu) (net 2))
-  (segment (start 108.700002 72.450002) (end 166.450002 72.450002) (width 0.25) (layer B.Cu) (net 2))
-  (segment (start 102.75 66.5) (end 108.700002 72.450002) (width 0.25) (layer B.Cu) (net 2))
-  (segment (start 102.75 61.5) (end 102.75 66.5) (width 0.25) (layer B.Cu) (net 2))
-  (segment (start 105 59.25) (end 102.75 61.5) (width 0.25) (layer B.Cu) (net 2))
-  (segment (start 105 55.886398) (end 105 59.25) (width 0.25) (layer B.Cu) (net 2))
-  (segment (start 97.25 48.136398) (end 105 55.886398) (width 0.25) (layer B.Cu) (net 2))
-  (via (at 144.5 69.75) (size 0.6) (drill 0.4) (layers F.Cu B.Cu) (net 2))
-  (via (at 149.25 74.5) (size 0.6) (drill 0.4) (layers F.Cu B.Cu) (net 2))
-  (via (at 162.25 69.75) (size 0.6) (drill 0.4) (layers F.Cu B.Cu) (net 2))
-  (via (at 158.25 69.75) (size 0.6) (drill 0.4) (layers F.Cu B.Cu) (net 2))
-  (via (at 141 69.75) (size 0.6) (drill 0.4) (layers F.Cu B.Cu) (net 2))
-  (via (at 130.25 74.5) (size 0.6) (drill 0.4) (layers F.Cu B.Cu) (net 2))
-  (via (at 125.25 69.75) (size 0.6) (drill 0.4) (layers F.Cu B.Cu) (net 2))
-  (via (at 126.75 74.5) (size 0.6) (drill 0.4) (layers F.Cu B.Cu) (net 2))
-  (via (at 122.5 69.75) (size 0.6) (drill 0.4) (layers F.Cu B.Cu) (net 2))
-  (via (at 153.75 117) (size 0.6) (drill 0.4) (layers F.Cu B.Cu) (net 2))
-  (via (at 159 106) (size 0.6) (drill 0.4) (layers F.Cu B.Cu) (net 2))
-  (via (at 158.75 92.25) (size 0.6) (drill 0.4) (layers F.Cu B.Cu) (net 2))
-  (via (at 145.75 74.5) (size 0.6) (drill 0.4) (layers F.Cu B.Cu) (net 2))
-  (via (at 146.25 116.75) (size 0.6) (drill 0.4) (layers F.Cu B.Cu) (net 2))
-  (via (at 141.25 108.75) (size 0.6) (drill 0.4) (layers F.Cu B.Cu) (net 2))
-  (via (at 141.25 92.25) (size 0.6) (drill 0.4) (layers F.Cu B.Cu) (net 2))
   (segment (start 165.5 115.75) (end 165.5 114.5) (width 0.25) (layer B.Cu) (net 2))
   (via (at 164.75 113.75) (size 0.6) (drill 0.4) (layers F.Cu B.Cu) (net 2))
